Commit message: 为了小车能够移动，修改小车轮子参数，以及导航的控制器

File: src/rm_nav_bringup/urdf/sentry_robot_sim.xacro (robot description, xacro)
@@ -110,9 +110,10 @@
     <parent link="base_link"/>
     <child link="wheel_1"/>
-    <origin rpy="${-PI/2} 0 0" xyz="0.1 0.13 0"/>
-    <axis xyz="0 0 1" />
+    <limit effort="100" velocity="100" />
+    <origin xyz="0.1 0.13 0"/>
+    <axis xyz="0 1 0" />
   </joint>
   <joint name="base_to_wheel2" type="continuous">
-    <axis xyz="0 0 1" />
+    <axis xyz="0 1 0" />
     <anchor xyz="0 0 0" />
     <limit effort="100" velocity="100" />
@@ -123,11 +124,12 @@
   <joint name="base_to_wheel3" type="continuous">
     <parent link="base_link"/>
-    <axis xyz="0 0 1" />
+    <axis xyz="0 1 0" />
     <child link="wheel_3"/>
-    <origin rpy="${-PI/2} 0 0" xyz="0.1 -0.13 0"/>
+    <limit effort="100" velocity="100" />
+    <origin xyz="0.1 -0.13 0"/>
   </joint>
   <joint name="base_to_wheel4" type="continuous">
     <parent link="base_link"/>
-    <axis xyz="0 0 1" />
+    <axis xyz="0 1 0" />
     <child link="wheel_4"/>
     <origin rpy="${-PI/2} 0 0" xyz="-0.1 -0.13 0"/>
@@ -191,9 +193,9 @@
       <ros>
         <namespace>/</namespace>
+        <remapping>cmd_vel:=cmd_vel</remapping>
+        <remapping>odom:=odom</remapping>
       </ros>
       <left_joint>base_to_wheel1</left_joint>
-      <left_joint>base_to_wheel2</left_joint>
       <right_joint>base_to_wheel3</right_joint>
-      <right_joint>base_to_wheel4</right_joint>
       <wheel_separation>0.26</wheel_separation>
       <wheel_radius>0.06</wheel_radius>
