Commit message: Use base_footprint as robot base frame

File: src/rm_nav_bringup/urdf/sentry_robot_real.xacro (robot description, xacro)
@@ -32,4 +32,10 @@
     <xacro:default_inertial mass="8.2"/>
   </link>
+  <link name="base_footprint"/>
+  <joint name="base_footprint_joint" type="fixed">
+    <parent link="base_footprint"/>
+    <child link="base_link"/>
+    <origin xyz="0 0 0" rpy="0 0 0"/>
+  </joint>
   <link name="wheel_1">
     <visual>

File: src/rm_nav_bringup/urdf/sentry_robot_sim.xacro (robot description, xacro)
@@ -33,7 +33,13 @@
     <xacro:default_inertial mass="8.2"/>
   </link>
+  <link name="base_footprint"/>
+  <joint name="base_footprint_joint" type="fixed">
+    <parent link="base_footprint"/>
+    <child link="base_link"/>
+    <origin xyz="0 0 0" rpy="0 0 0"/>
+  </joint>
   <joint name="dummy_joint" type="fixed">
      <parent link="dummy"/>
-     <child link="base_link"/>
+     <child link="base_footprint"/>
   </joint>
   <link name="wheel_1">

File: src/rm_simulation/pb_rm_simulation/urdf/simulation_waking_robot.xacro (robot description, xacro)
@@ -33,7 +33,13 @@
     <xacro:default_inertial mass="8.2"/>
   </link>
+  <link name="base_footprint"/>
+  <joint name="base_footprint_joint" type="fixed">
+    <parent link="base_footprint"/>
+    <child link="base_link"/>
+    <origin xyz="0 0 0" rpy="0 0 0"/>
+  </joint>
   <joint name="dummy_joint" type="fixed">
      <parent link="dummy"/>
-     <child link="base_link"/>
+     <child link="base_footprint"/>
   </joint>
   <link name="wheel_1">
